File: schematic/LED_DISPLAY_BOARD.kicad_sch (KiCad schematic)
At the start: 23 parts, among them J1 Conn_01x27, U1 SM420561N, U2 SM420561N, U3 SM420561N, U4 SM420561N

Commit message: mit license update
Other:
- company: JDC -> sparkletron
Changed lines of the file:
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@@
     (date "2022-12-11")
     (rev "v1.0")
-    (company "JDC")
+    (company "sparkletron")
+    (comment 1 "Jay Convertino")
+    (comment 2 "MIT License")
   )
   (junction (at 205.74 104.775) (diameter 0) (color 0 0 0 0)
