File: schematic/Mil_Time_Clock.kicad_sch (KiCad schematic)
At the start: 0 parts

Commit message: mit license update
Other:
- company: JDC -> sparkletron
Changed lines of the file:
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@@
     (date "2022-12-11")
     (rev "v1.0")
-    (company "JDC")
+    (company "sparkletron")
+    (comment 1 "Jay Convertino")
+    (comment 2 "MIT License")
   )
   (wire (pts (xy 131.445 80.01) (xy 148.59 80.01))
